File: Hardware/xva1-ui/xva1-ui.kicad_pcb (KiCad board)
At the start: 2 copper layers, 285 x 130 mm, 55 parts, among them J1 DIN-5_180degree, J2 DIN-5_180degree, J3 DIN-5_180degree, J4 Conn_01x02, J5 Conn_01x02, J6 Conn_01x02, SW0 Rotary Encoder, SW1 Rotary Encoder, SW10 SW_Push, SW11 SW_Push, SW12 SW_Push, SW13 SW_Push_LED, SW14 SW_Push_LED, SW15 SW_Push_LED, SW16 SW_Push_LED, SW17 SW_Push_LED, SW18 SW_Push_LED, SW19 SW_Push_LED, SW2 Rotary Encoder, SW20 SW_Push_LED, SW21 SW_Push_LED, SW22 SW_Push_LED, SW3 Rotary Encoder, SW4 Rotary Encoder, SW5 Rotary Encoder, SW6 Rotary Encoder, SW7 Rotary Encoder, SW8 Rotary Encoder, SW9 SW_Push, U1 Seeeduino XIAO, U2 MCP23017, U3 MCP23017, U4 MCP23017, U5 TCA9548A, U6 CMOD-A7, U7 UDA1334, U8 24LC1025, U9 4N36

Commit message: Updated PCB layout + Added Gerber files
Parts:
- added R10: 470, Resistor_THT:R_Axial_DIN0207_L6.3mm_D2.5mm_P10.16mm_Horizontal, F.Cu at (266.5, 82.2)
- added R11: 470, Resistor_THT:R_Axial_DIN0207_L6.3mm_D2.5mm_P10.16mm_Horizontal, F.Cu at (283.1, 82.2)
- added R12: 470, Resistor_THT:R_Axial_DIN0207_L6.3mm_D2.5mm_P10.16mm_Horizontal, F.Cu at (233.3, 140.8)
- added R13: 470, Resistor_THT:R_Axial_DIN0207_L6.3mm_D2.5mm_P10.16mm_Horizontal, F.Cu at (249.9, 140.8)
- added R14: 470, Resistor_THT:R_Axial_DIN0207_L6.3mm_D2.5mm_P10.16mm_Horizontal, F.Cu at (266.5, 140.8)
- added R15: 470, Resistor_THT:R_Axial_DIN0207_L6.3mm_D2.5mm_P10.16mm_Horizontal, F.Cu at (283.1, 140.8)
- added R6: 470, Resistor_THT:R_Axial_DIN0207_L6.3mm_D2.5mm_P10.16mm_Horizontal, F.Cu at (207.6, 82.2)
- added R7: 470, Resistor_THT:R_Axial_DIN0207_L6.3mm_D2.5mm_P10.16mm_Horizontal, F.Cu at (207.6, 140.8)
- added R8: 470, Resistor_THT:R_Axial_DIN0207_L6.3mm_D2.5mm_P10.16mm_Horizontal, F.Cu at (233.3, 82.2)
- added R9: 470, Resistor_THT:R_Axial_DIN0207_L6.3mm_D2.5mm_P10.16mm_Horizontal, F.Cu at (249.9, 82.2)
- U8: value 24LC1025 -> 24LC1025-I/P
- moved REF** 1.80 mm to (11.1, 25.5)
- moved REF** 1.50 mm to (287.1, 25.5)
- moved REF** 1.00 mm to (11.1, 146.0)
- moved U1 1.00 mm to (16.2, 45.4)
Connections:
- SW13 pad 4: LED-UP -> Net-(R6-Pad1)
- SW14 pad 4: LED-DWN -> Net-(R7-Pad1)
- SW15 pad 4: LED-SC1 -> Net-(R8-Pad1)
- SW16 pad 4: LED-SC2 -> Net-(R9-Pad1)
- SW17 pad 4: LED-SC3 -> Net-(R10-Pad1)
- SW18 pad 4: LED-SC4 -> Net-(R11-Pad1)
- SW19 pad 4: LED-SC5 -> Net-(R12-Pad1)
- SW20 pad 4: LED-SC6 -> Net-(R13-Pad1)
- SW21 pad 4: LED-SC7 -> Net-(R14-Pad1)
- SW22 pad 4: LED-SC8 -> Net-(R15-Pad1)
Routing:
- net GND: track 62.3 -> 27.1 mm
- net LED-UP: track 64.0 -> 42.3 mm
- net Net-(R15-Pad1): track 0.00 -> 18.8 mm
- net Net-(R6-Pad1): track 0.00 -> 17.5 mm
- net Net-(R8-Pad1): track 0.00 -> 17.2 mm
- net Net-(R10-Pad1): track 0.00 -> 17.2 mm
- net Net-(R9-Pad1): track 0.00 -> 17.1 mm
- net Net-(R11-Pad1): track 0.00 -> 17.1 mm
- net Net-(R7-Pad1): track 0.00 -> 16.1 mm
- net Net-(R14-Pad1): track 0.00 -> 16.1 mm
- net Net-(R13-Pad1): track 0.00 -> 16.0 mm
- net Net-(R12-Pad1): track 0.00 -> 15.9 mm
- net LED-SC2: track 74.6 -> 59.0 mm
- net LED-SC4: track 98.3 -> 83.4 mm
- net LED-SC5: track 82.3 -> 97.1 mm
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Other:
- board size 285 x 130 mm -> 284 x 128.5 mm
- board text added: "24LC1025"

Commit message: Changed mounting holes + board outline
Parts:
- removed the REF** at (215.1, 85.0)
- removed the REF** at (82.1, 85.0)
- removed the REF** at (287.1, 146.0)
- removed the REF** at (287.1, 25.5)
- removed the REF** at (11.1, 25.5)
- removed the REF** at (11.1, 146.0)
- added REF**: Kosmo_Panel_Mounting_Hole, Kosmo_panel:Kosmo_Panel_Mounting_Hole, F.Cu at (82.0, 85.8)
- added REF**: Kosmo_Panel_Mounting_Hole, Kosmo_panel:Kosmo_Panel_Mounting_Hole, F.Cu at (216.0, 85.8)
- added REF**: Kosmo_Panel_Mounting_Hole, Kosmo_panel:Kosmo_Panel_Mounting_Hole, F.Cu at (288.0, 147.0)
- added REF**: Kosmo_Panel_Mounting_Hole, Kosmo_panel:Kosmo_Panel_Mounting_Hole, F.Cu at (288.0, 24.5)
- added REF**: Kosmo_Panel_Mounting_Hole, Kosmo_panel:Kosmo_Panel_Mounting_Hole, F.Cu at (10.0, 24.5)
- added REF**: Kosmo_Panel_Mounting_Hole, Kosmo_panel:Kosmo_Panel_Mounting_Hole, F.Cu at (10.0, 147.0)
